File: FishingReelController.brd (EAGLE design)
At the start: 160 x 100 mm, 33 parts, among them Q1 NVF6P02, U1 TRINKETPRO, U2 MCP4921

Commit message: backup
Parts:
- added R13, R14, R15, R16, R17: (no value), GradeFreeEngineer:R0603(1608)
- moved SJ2 225.1 mm to (-11.4, 64.8), turned to 90 degrees
- moved C3 223.5 mm to (-26.7, 52.1), turned to 270 degrees
- moved SJ1 219.8 mm to (-29.2, 64.8), turned to 90 degrees
- moved C2 219.7 mm to (-25.4, 52.1), turned to 270 degrees
- moved R12 209.8 mm to (-15.2, 59.7)
- moved C1 209.6 mm to (-19.1, 45.7), turned to 180 degrees
- moved TR3 208.5 mm to (-15.2, 64.8), turned to 90 degrees
- moved JP3 198.1 mm to (30.5, 53.3), turned to 90 degrees
- moved JP2 187.0 mm to (-30.5, 53.3), turned to 270 degrees
- moved R11 168.2 mm to (-11.4, 39.4)
- moved R10 167.0 mm to (-11.4, 41.9)
- moved R9 165.7 mm to (-11.4, 44.5)
- moved R8 155.6 mm to (-11.4, 38.1), turned to 180 degrees
- moved R7 154.3 mm to (-11.4, 40.6), turned to 180 degrees
- moved R6 153.0 mm to (-11.4, 43.2), turned to 180 degrees
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Connections:
- new net N$7: R13.1, U1.7
- net DGND: now also R16.1, R17.1
- net MODE_A: now also U1.9
- net MODE_B: now also U1.10
- net OK_STOP: now also U1.11
- net PICKUP: now also U1.1
- net POTEN_ADC: now also R13.2; no longer U1.7
- net POTEN_DAC: now also R14.1, R15.1, R16.2, R17.2
- net SHIPREEL_POWER: now also R14.2, R15.2
Other:
- board size 160 x 100 mm -> 17.8 x 37.3 mm

Commit message: gerber done
Parts:
- added LOGO1: GRADEFREELOGO-20, GradeFreeEngineer:GRADEFREELOGO-20
- added TVS1: SD15C, berry:SOD-323-NOPOL
- added X1, X5: 5268-02, OSSI:5628-02
- moved H2 259.1 mm to (33.0, 77.0)
- moved H1 255.0 mm to (-33.0, 77.0)
- moved H4 195.4 mm to (33.0, 3.00)
- moved H3 190.0 mm to (-33.0, 3.00)
- moved SJ1 9.53 mm to (-21.6, 70.5), turned to 0 degrees
- moved S3 3.49 mm to (20.0, 12.0)
- moved S2 3.13 mm to (-20.0, 12.0)
- moved R3 2.62 mm to (-21.6, 60.3)
- moved S1 1.78 mm to (-20.0, 30.0)
- moved Q1 1.27 mm to (-21.6, 64.8)
- moved R12 0.64 mm to (-15.2, 60.3)
- turned R13 to 180 degrees
Connections:
- new net +12V: TVS1.2, U1.24, X1.1, X5.1
- net DGND: now also TVS1.1, X1.2, X5.2
Routing:
- net VCC: track 0.00 -> 206.8 mm, vias 0 -> 4
- net +12V: track 0.00 -> 81.6 mm
- net N$18: track 0.00 -> 65.2 mm, vias 0 -> 2
- net N$17: track 0.00 -> 48.9 mm, vias 0 -> 2
- net N$16: track 0.00 -> 34.5 mm
- net DGND: track 0.00 -> 33.3 mm, vias 0 -> 10
- net SHIPREEL_POWER: track 0.00 -> 28.2 mm
- net PICKUP_SW: track 0.00 -> 24.9 mm
- net POTEN_DAC: track 0.00 -> 24.4 mm, vias 0 -> 1
- net ENC2_PULSE: track 0.00 -> 20.4 mm
- net ENC1_PULSE: track 0.00 -> 20.4 mm
- net DAC_CS: track 0.00 -> 19.7 mm
- net POTEN_ADC: track 0.00 -> 18.3 mm
- net N$6: track 0.00 -> 15.3 mm, vias 0 -> 2
- net START_SW: track 0.00 -> 15.0 mm
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- added copper zone on layer 16, net DGND
Other:
- board size 17.8 x 37.3 mm -> 72 x 80 mm
- board text added: "Electric Reel"
- board text added: "Fishing Action"
- board text added: "controller ver 0.1"
