File: FishingReelController.sch (EAGLE design)
At the start: 33 parts, among them Q1 NVF6P02, U1 TRINKETPRO, U2 MCP4921

Commit message: backup
Parts:
- added R13, R14, R15, R16, R17: (no value), GradeFreeEngineer:R0603(1608)
Connections:
- new net N$7: R13.1, U1.A0
- net DGND: now also R16.1, R17.1
- net MODE_A: now also U1.A2
- net MODE_B: now also U1.A3
- net OK_STOP: now also U1.A4
- net PICKUP: now also U1.D9
- net POTEN_ADC: now also R13.2; no longer U1.A0
- net POTEN_DAC: now also R14.1, R15.1, R16.2, R17.2
- net SHIPREEL_POWER: now also R14.2, R15.2
Changed lines of the file:
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@@
 <part name="H3" library="berry" deviceset="MOUNT-PAD-ROUND" device="3.2"/>
 <part name="H4" library="berry" deviceset="MOUNT-PAD-ROUND" device="3.2"/>
+<part name="R13" library="GradeFreeEngineer" deviceset="R" device="0603(1608)"/>
+<part name="R14" library="GradeFreeEngineer" deviceset="R" device="0603(1608)"/>
+<part name="R15" library="GradeFreeEngineer" deviceset="R" device="0603(1608)"/>
+<part name="R16" library="GradeFreeEngineer" deviceset="R" device="0603(1608)"/>
+<part name="R17" library="GradeFreeEngineer" deviceset="R" device="0603(1608)"/>
+<part name="GND17" library="GradeFreeEngineer" deviceset="DGND" device=""/>
 </parts>
 <sheets>
@@
 <instance part="H3" gate="G$1" x="114.3" y="-17.78"/>
 <instance part="H4" gate="G$1" x="157.48" y="-17.78"/>
+<instance part="R13" gate="G$1" x="25.4" y="50.8" rot="R180"/>
+<instance part="R14" gate="G$1" x="119.38" y="147.32" rot="R90"/>
+<instance part="R15" gate="G$1" x="127" y="147.32" rot="R90"/>
+<instance part="R16" gate="G$1" x="119.38" y="121.92" rot="R90"/>
+<instance part="R17" gate="G$1" x="127" y="121.92" rot="R90"/>
+<instance part="GND17" gate="1" x="127" y="111.76"/>
 </instances>
 <busses>
@@
 <pinref part="C1" gate="G$1" pin="2"/>
 <wire x1="106.68" y1="157.48" x2="101.6" y2="157.48" width="0.1524" layer="91"/>
+</segment>
+<segment>
+<pinref part="GND17" gate="1" pin="DGND"/>
+<pinref part="R17" gate="G$1" pin="1"/>
+<wire x1="127" y1="114.3" x2="127" y2="116.84" width="0.1524" layer="91"/>
+<pinref part="R16" gate="G$1" pin="1"/>
+<wire x1="127" y1="114.3" x2="119.38" y2="114.3" width="0.1524" layer="91"/>
+<wire x1="119.38" y1="114.3" x2="119.38" y2="116.84" width="0.1524" layer="91"/>
+<junction x="127" y="114.3"/>
 </segment>
 </net>
@@
 <label x="200.66" y="66.04" size="1.778" layer="95" rot="R180" xref="yes"/>
 </segment>
+<segment>
+<pinref part="U1" gate="G$1" pin="A4"/>
+<wire x1="33.02" y1="40.64" x2="27.94" y2="40.64" width="0.1524" layer="91"/>
+<label x="27.94" y="40.64" size="1.778" layer="95" rot="R180" xref="yes"/>
+</segment>
 </net>
 <net name="MODE_B" class="0">
@@
 <label x="177.8" y="66.04" size="1.778" layer="95" rot="R180" xref="yes"/>
 </segment>
+<segment>
+<pinref part="U1" gate="G$1" pin="A3"/>
+<wire x1="33.02" y1="43.18" x2="27.94" y2="43.18" width="0.1524" layer="91"/>
+<label x="27.94" y="43.18" size="1.778" layer="95" rot="R180" xref="yes"/>
+</segment>
 </net>
 <net name="MODE_A" class="0">
@@
 <wire x1="157.48" y1="66.04" x2="154.94" y2="66.04" width="0.1524" layer="91"/>
 <label x="154.94" y="66.04" size="1.778" layer="95" rot="R180" xref="yes"/>
+</segment>
+<segment>
+<pinref part="U1" gate="G$1" pin="A2"/>
+<wire x1="33.02" y1="45.72" x2="27.94" y2="45.72" width="0.1524" layer="91"/>
+<label x="27.94" y="45.72" size="1.778" layer="95" rot="R180" xref="yes"/>
 </segment>
 </net>
@@
 <junction x="45.72" y="142.24"/>
 </segment>
+<segment>
+<pinref part="R14" gate="G$1" pin="2"/>
+<wire x1="119.38" y1="152.4" x2="119.38" y2="154.94" width="0.1524" layer="91"/>
+<pinref part="R15" gate="G$1" pin="2"/>
+<wire x1="119.38" y1="154.94" x2="127" y2="154.94" width="0.1524" layer="91"/>
+<wire x1="127" y1="154.94" x2="127" y2="152.4" width="0.1524" layer="91"/>
+<wire x1="127" y1="154.94" x2="127" y2="157.48" width="0.1524" layer="91"/>
+<junction x="127" y="154.94"/>
+<label x="127" y="157.48" size="1.778" layer="95" rot="R90" xref="yes"/>
+</segment>
 </net>
 <net name="ROCKREEL_POWER" class="0">
@@
 <segment>
 <pinref part="U2" gate="G$1" pin="DACA"/>
-<wire x1="101.6" y1="134.62" x2="114.3" y2="134.62" width="0.1524" layer="91"/>
-<label x="114.3" y="134.62" size="1.778" layer="95" xref="yes"/>
+<wire x1="101.6" y1="134.62" x2="124.46" y2="134.62" width="0.1524" layer="91"/>
+<label x="132.08" y="134.62" size="1.778" layer="95" xref="yes"/>
+<pinref part="R16" gate="G$1" pin="2"/>
+<wire x1="124.46" y1="134.62" x2="132.08" y2="134.62" width="0.1524" layer="91"/>
+<wire x1="119.38" y1="127" x2="119.38" y2="129.54" width="0.1524" layer="91"/>
+<pinref part="R17" gate="G$1" pin="2"/>
+<wire x1="119.38" y1="129.54" x2="124.46" y2="129.54" width="0.1524" layer="91"/>
+<wire x1="124.46" y1="129.54" x2="127" y2="129.54" width="0.1524" layer="91"/>
+<wire x1="127" y1="129.54" x2="127" y2="127" width="0.1524" layer="91"/>
+<wire x1="124.46" y1="129.54" x2="124.46" y2="134.62" width="0.1524" layer="91"/>
+<junction x="124.46" y="129.54"/>
+<junction x="124.46" y="134.62"/>
+<pinref part="R14" gate="G$1" pin="1"/>
+<wire x1="119.38" y1="142.24" x2="119.38" y2="139.7" width="0.1524" layer="91"/>
+<pinref part="R15" gate="G$1" pin="1"/>
+<wire x1="119.38" y1="139.7" x2="124.46" y2="139.7" width="0.1524" layer="91"/>
+<wire x1="124.46" y1="139.7" x2="127" y2="139.7" width="0.1524" layer="91"/>
+<wire x1="127" y1="139.7" x2="127" y2="142.24" width="0.1524" layer="91"/>
+<wire x1="124.46" y1="134.62" x2="124.46" y2="139.7" width="0.1524" layer="91"/>
+<junction x="124.46" y="139.7"/>
 </segment>
 </net>
@@
 </segment>
 <segment>
-<pinref part="U1" gate="G$1" pin="A0"/>
-<wire x1="33.02" y1="50.8" x2="27.94" y2="50.8" width="0.1524" layer="91"/>
-<label x="27.94" y="50.8" size="1.778" layer="95" rot="R180" xref="yes"/>
+<pinref part="R13" gate="G$1" pin="2"/>
+<wire x1="20.32" y1="50.8" x2="15.24" y2="50.8" width="0.1524" layer="91"/>
+<label x="15.24" y="50.8" size="1.778" layer="95" rot="R180" xref="yes"/>
 </segment>
 </net>
@@
 <label x="15.24" y="114.3" size="1.778" layer="95" rot="R180" xref="yes"/>
 </segment>
+<segment>
+<pinref part="U1" gate="G$1" pin="D9"/>
+<wire x1="33.02" y1="66.04" x2="27.94" y2="66.04" width="0.1524" layer="91"/>
+<label x="27.94" y="66.04" size="1.778" layer="95" rot="R180" xref="yes"/>
+</segment>
 </net>
 <net name="DAC_CS" class="0">
@@
 </segment>
 </net>
+<net name="N$7" class="0">
+<segment>
+<pinref part="U1" gate="G$1" pin="A0"/>
+<pinref part="R13" gate="G$1" pin="1"/>
+<wire x1="33.02" y1="50.8" x2="30.48" y2="50.8" width="0.1524" layer="91"/>
+</segment>
+</net>

Commit message: gerber done
Parts:
- added LOGO1: GRADEFREELOGO-20, GradeFreeEngineer:GRADEFREELOGO-20
- added TVS1: SD15C, berry:SD0
- added X1, X5: 5268-02, OSSI:5268-02
Connections:
- new net +12V: TVS1.P$2, U1.VBAT, X1.1, X5.1
- net DGND: now also TVS1.P$1, X1.2, X5.2
Changed lines of the file:
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@@
 <part name="R17" library="GradeFreeEngineer" deviceset="R" device="0603(1608)"/>
 <part name="GND17" library="GradeFreeEngineer" deviceset="DGND" device=""/>
+<part name="X5" library="OSSI" deviceset="5268-02" device=""/>
+<part name="X1" library="OSSI" deviceset="5268-02" device=""/>
+<part name="GND18" library="GradeFreeEngineer" deviceset="DGND" device=""/>
+<part name="P+8" library="berry" deviceset="+12V" device=""/>
+<part name="TVS1" library="berry" deviceset="SD0" device="" value="SD15C"/>
+<part name="P+9" library="berry" deviceset="+12V" device=""/>
+<part name="LOGO1" library="GradeFreeEngineer" deviceset="GRADEFREELOGO" device="-20"/>
 </parts>
 <sheets>
@@
 <instance part="R17" gate="G$1" x="127" y="121.92" rot="R90"/>
 <instance part="GND17" gate="1" x="127" y="111.76"/>
+<instance part="X5" gate="G$1" x="-40.64" y="139.7" rot="R90"/>
+<instance part="X1" gate="G$1" x="-20.32" y="139.7" rot="R90"/>
+<instance part="GND18" gate="1" x="-43.18" y="111.76"/>
+<instance part="P+8" gate="1" x="-12.7" y="129.54" rot="R270"/>
+<instance part="TVS1" gate="G$1" x="-33.02" y="119.38" rot="R90"/>
+<instance part="P+9" gate="1" x="66.04" y="76.2"/>
+<instance part="LOGO1" gate="G$1" x="-30.48" y="198.12"/>
 </instances>
 <busses>
@@
 <wire x1="119.38" y1="114.3" x2="119.38" y2="116.84" width="0.1524" layer="91"/>
 <junction x="127" y="114.3"/>
+</segment>
+<segment>
+<pinref part="X5" gate="G$1" pin="2"/>
+<wire x1="-43.18" y1="134.62" x2="-43.18" y2="114.3" width="0.1524" layer="91"/>
+<pinref part="X1" gate="G$1" pin="2"/>
+<wire x1="-43.18" y1="114.3" x2="-33.02" y2="114.3" width="0.1524" layer="91"/>
+<wire x1="-33.02" y1="114.3" x2="-22.86" y2="114.3" width="0.1524" layer="91"/>
+<wire x1="-22.86" y1="114.3" x2="-22.86" y2="134.62" width="0.1524" layer="91"/>
+<pinref part="GND18" gate="1" pin="DGND"/>
+<junction x="-43.18" y="114.3"/>
+<pinref part="TVS1" gate="G$1" pin="P$1"/>
+<junction x="-33.02" y="114.3"/>
 </segment>
 </net>
@@
 </segment>
 </net>
+<net name="+12V" class="0">
+<segment>
+<pinref part="X5" gate="G$1" pin="1"/>
+<wire x1="-40.64" y1="134.62" x2="-40.64" y2="129.54" width="0.1524" layer="91"/>
+<pinref part="X1" gate="G$1" pin="1"/>
+<wire x1="-40.64" y1="129.54" x2="-33.02" y2="129.54" width="0.1524" layer="91"/>
+<wire x1="-33.02" y1="129.54" x2="-20.32" y2="129.54" width="0.1524" layer="91"/>
+<wire x1="-20.32" y1="129.54" x2="-20.32" y2="134.62" width="0.1524" layer="91"/>
+<pinref part="P+8" gate="1" pin="+12V"/>
+<wire x1="-20.32" y1="129.54" x2="-15.24" y2="129.54" width="0.1524" layer="91"/>
+<junction x="-20.32" y="129.54"/>
+<pinref part="TVS1" gate="G$1" pin="P$2"/>
+<junction x="-33.02" y="129.54"/>
+</segment>
+<segment>
+<pinref part="U1" gate="G$1" pin="VBAT"/>
+<wire x1="63.5" y1="66.04" x2="66.04" y2="66.04" width="0.1524" layer="91"/>
+<wire x1="66.04" y1="66.04" x2="66.04" y2="73.66" width="0.1524" layer="91"/>
+<pinref part="P+9" gate="1" pin="+12V"/>
+</segment>
+</net>
