File: SmartLURE.brd (EAGLE design)
At the start: 15.2 x 34.3 mm, 22 parts, among them U1 TRINKET

Commit message: gerber done
Parts:
- added LOGO1: GRADEFREELOGO-10, GradeFreeEngineer:GRADEFREELOGO-10
Other:
- board text added: "Smart Lure"
- board text added: "ver 0.1"
Changed lines of the file:
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@@
 <layer number="19" name="Unrouted" color="6" fill="1" visible="yes" active="yes"/>
 <layer number="20" name="Dimension" color="15" fill="1" visible="yes" active="yes"/>
-<layer number="21" name="tPlace" color="7" fill="1" visible="yes" active="yes"/>
+<layer number="21" name="tPlace" color="7" fill="1" visible="no" active="yes"/>
 <layer number="22" name="bPlace" color="7" fill="1" visible="no" active="yes"/>
 <layer number="23" name="tOrigins" color="15" fill="1" visible="yes" active="yes"/>
@@
 <layer number="27" name="tValues" color="7" fill="1" visible="no" active="yes"/>
 <layer number="28" name="bValues" color="7" fill="1" visible="no" active="yes"/>
-<layer number="29" name="tStop" color="7" fill="3" visible="no" active="yes"/>
+<layer number="29" name="tStop" color="7" fill="3" visible="yes" active="yes"/>
 <layer number="30" name="bStop" color="7" fill="6" visible="no" active="yes"/>
 <layer number="31" name="tCream" color="7" fill="4" visible="no" active="yes"/>
@@
 <hole x="6.7675" y="1.27" drill="0.7"/>
 <hole x="-6.7675" y="1.27" drill="0.7"/>
+<text x="-4.1275" y="29.21" size="0.8128" layer="1" font="vector">Smart Lure</text>
+<text x="-4.1275" y="29.21" size="0.8128" layer="29" font="vector">Smart Lure</text>
+<text x="-4.1275" y="27.94" size="0.8128" layer="1" font="vector">ver 0.1</text>
+<text x="-4.1275" y="27.94" size="0.8128" layer="29" font="vector">ver 0.1</text>
 </plain>
 <attributes>
@@
 <attribute name="VALUE" x="7.62" y="9.525" size="1.27" layer="28" rot="MR0"/>
 </element>
+<element name="LOGO1" library="GradeFreeEngineer" package="GRADEFREELOGO-10" value="GRADEFREELOGO-10" x="-3.81" y="30.48"/>
 </elements>
 <signals>
