File: SmartLURE.sch (EAGLE design)
At the start: 22 parts, among them U1 TRINKET

Commit message: gerber done
Parts:
- added LOGO1: GRADEFREELOGO-10, GradeFreeEngineer:GRADEFREELOGO-10
Changed lines of the file:
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@@
 <part name="JP4" library="adafruit" deviceset="PINHD-1X1" device="CB"/>
 <part name="JP5" library="adafruit" deviceset="PINHD-1X1" device="CB"/>
+<part name="LOGO1" library="GradeFreeEngineer" deviceset="GRADEFREELOGO" device="-10"/>
 </parts>
 <sheets>
@@
 <instance part="JP4" gate="G$1" x="208.28" y="101.6" rot="R180"/>
 <instance part="JP5" gate="G$1" x="208.28" y="96.52" rot="R180"/>
+<instance part="LOGO1" gate="G$1" x="43.18" y="33.02"/>
 </instances>
 <busses>
